File: ai03-pcb-guide.kicad_pcb (KiCad board)
At the start: 2 copper layers, 24 parts, among them SW1 SW_Push, U1 ATmega32U4-AU, Y1 16MHz

Commit message: complete
Routing:
- net Net-(USB1-Pad6): track 0.00 -> 17.3 mm
- added copper zone on B.Cu, net GND

Commit message: complete
Other:
- board outline added: 89.8 x 38.3 mm
